File: kicad/boards/main/main.kicad_pcb (KiCad board)
At the start: 2 copper layers, 160 x 100 mm, 4 parts

Commit message: Commit what I've got so far
Parts:
- removed MH1: MountingHole_2.7mm_M2.5_DIN965, MountingHole:MountingHole_2.7mm_M2.5_DIN965
- added J1: DIN41612_03x32_C_Split, Connector_DIN:DIN41612_C_3x32_Male_Horizontal_THT, F.Cu at (209.7, 55.7)
- added J2: Barrel_Jack_Switch, Package_DFN_QFN:QFN-40-1EP_6x6mm_P0.5mm_EP4.6x4.6mm, F.Cu at (40.5, 10.2)
- added J3: P2_edge_connector, gauntlet:4UCON_10156_2x40_P1.27mm_Socket_Horizontal, F.Cu at (196.0, 53.2)
- added SW1: SW_SPDT, Button_Switch_THT:SW_NKK_GW12LJP, F.Cu at (38.0, 1.50)
- added U2: PocketBeagle, Module:BeagleBoard_PocketBeagle, F.Cu at (3.81, 7.58)
Routing:
- net /SMART_OUT15: track 0.00 -> 17.6 mm
- net /SMART_OUT13: track 0.00 -> 15.3 mm
- net /SMART_OUT14: track 0.00 -> 14.4 mm
- net /SMART_OUT11: track 0.00 -> 13.1 mm
- net /SMART_OUT1: track 0.00 -> 13.1 mm
- net /SMART_OUT9: track 0.00 -> 12.1 mm
- net /SMART_OUT3: track 0.00 -> 12.1 mm
- net /SMART_OUT0: track 0.00 -> 11.8 mm
- net /SMART_OUT12: track 0.00 -> 11.8 mm
- net /SMART_OUT7: track 0.00 -> 11.0 mm
- net /SMART_OUT5: track 0.00 -> 11.0 mm
- net /SMART_OUT10: track 0.00 -> 10.7 mm
- net /SMART_OUT2: track 0.00 -> 10.7 mm
- net /SMART_OUT8: track 0.00 -> 9.66 mm
- net /SMART_OUT4: track 0.00 -> 9.66 mm
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