File: kicad/boards/main/main.kicad_sch (KiCad schematic)
At the start: 1 part, among them J1 DIN41612_03x32_C_Split

Commit message: Commit what I've got so far
Parts:
- added J2: Barrel_Jack_Switch, Package_DFN_QFN:QFN-40-1EP_6x6mm_P0.5mm_EP4.6x4.6mm, symbol Connector:Barrel_Jack_Switch
- added J3: P2_edge_connector, gauntlet:4UCON_10156_2x40_P1.27mm_Socket_Horizontal, symbol p2_edge_connector:P2_edge_connector
- added SW1: SW_SPDT, Button_Switch_THT:SW_NKK_GW12LJP, symbol Switch:SW_SPDT
- added U2: PocketBeagle, Module:BeagleBoard_PocketBeagle, symbol MCU_Module:PocketBeagle
Connections:
- net SMART_IN0: now also J3.80 (P38)
- net SMART_IN1: now also J3.79 (P39)
- net SMART_IN10: now also J3.70 (P46)
- net SMART_IN11: now also J3.69 (P47)
- net SMART_IN12: now also J3.68 (V24_31)
- net SMART_IN13: now also J3.67 (V48_55)
- net SMART_IN14: now also J3.66 (P48)
- net SMART_IN15: now also J3.65 (P49)
- net SMART_IN2: now also J3.78 (V32_39)
- net SMART_IN3: now also J3.77 (V40_47)
- net SMART_IN4: now also J3.76 (P40)
- net SMART_IN5: now also J3.75 (P41)
- net SMART_IN6: now also J3.74 (P42)
- net SMART_IN7: now also J3.73 (P43)
- net SMART_IN8: now also J3.72 (P44)
- net SMART_IN9: now also J3.71 (P45)
- net SMART_OUT0: now also J3.9 (P31)
- net SMART_OUT1: now also J3.10 (P30)
- net SMART_OUT10: now also J3.19 (P21)
- net SMART_OUT11: now also J3.20 (P20)
- net SMART_OUT12: now also J3.21 (P19)
- net SMART_OUT13: now also J3.22 (P18)
- net SMART_OUT14: now also J3.23 (P17)
- net SMART_OUT15: now also J3.24 (P16)
- net SMART_OUT2: now also J3.11 (P29)
- net SMART_OUT3: now also J3.12 (P28)
- net SMART_OUT4: now also J3.13 (P27)
- net SMART_OUT5: now also J3.14 (P26)
- net SMART_OUT6: now also J3.15 (P25)
- net SMART_OUT7: now also J3.16 (P24)
- net SMART_OUT8: now also J3.17 (P23)
- net SMART_OUT9: now also J3.18 (P22)
- new net: U2.15 (GND), U2.16 (GND), U2.22 (GND), U2.51 (GND), U2.57 (GND)
- new net P2_RESETn: J3.46 (RESn)
